File: pwrcon_1.sch (KiCad schematic (older format))
At the start: 52 parts, among them J1 CON3, J4 CON3, J5 Conn_01x03_Female, J6 Conn_01x04, J7 CON3, J8 Conn_01x03_Female, Q1 Q_PNP_BEC, U1 LM358, U2 ISOW7841DWE, U3 THVD1500D, U4 SN74LV1T34DBVR, U5 SN74LV1T34DBVR, U6 SN74LV1T34DBVR, U7 MIC5219-3.3YMM

Commit message: More routing, component footprints finalised and missing ones added into repo
Parts:
- added TP5: TestPoint, TestPoint:TestPoint_Loop_D1.80mm_Drill1.0mm_Beaded, symbol Connector:TestPoint
- C4, C6, C8: MFG Name (none) -> Kemet; MFG Part Num (none) -> C0603C104J4RACTU
- C5, C7: MFG Name (none) -> Kemet; MFG Part Num (none) -> C0603C106M9PACTU
- D1: MFG Name (none) -> Diodes Inc; MFG Part Num (none) -> BAV16W-7-F
- D2: Manufacturer Multicomp / Littelfuse -> Multicomp / Diodes
- R1, R2, R6: MFG Name (none) -> Rohm; MFG Part Num (none) -> ESR03EZPJ102
- R10, R11: footprint Resistor_SMD:R_0603_1608Metric_Pad1.05x0.95mm_HandSolder -> Resistor_SMD:R_2512_6332Metric_Pad1.52x3.35mm_HandSolder; MFG Name (none) -> Vishay; MFG Part Num (none) -> CRCW251210R0FKEG
- R12: MFG Name (none) -> Vishay; MFG Part Num (none) -> CRCW0603120RJNEA
- R4: MFG Name (none) -> Vishay; MFG Part Num (none) -> RCS06031M00FKEA
- R5: MFG Name (none) -> Rohm; MFG Part Num (none) -> ESR03EZPJ472
- R8: footprint Resistor_SMD:R_0603_1608Metric_Pad1.05x0.95mm_HandSolder -> Resistor_SMD:R_0805_2012Metric_Pad1.15x1.40mm_HandSolder; MFG Name (none) -> Panasonic; MFG Part Num (none) -> ERJ-P06J472V
- R9: MFG Name (none) -> Rohm; MFG Part Num (none) -> ESR03EZPJ152
Connections:
- net at U2.11 (IND), U3.1 (R): now also TP4.1
- net at U2.12 (OUTC), U3.3 (DE): no longer TP4.1
- net at U2.14 (OUTA), U3.4 (D): now also TP5.1
Other:
- note added: "Continuity (NC) Check"
- note added: "Voltage Regulator"
- moved on the sheet: TP4
Changed lines of the file:
@@
 F 2 "Resistor_SMD:R_0603_1608Metric" H 1125 6050 50  0001 C CNN
 F 3 "~" H 1125 6050 50  0001 C CNN
+F 4 "Rohm" H 1125 6050 50  0001 C CNN "MFG Name"
+F 5 "ESR03EZPJ102" H 1125 6050 50  0001 C CNN "MFG Part Num"
 	1    1125 6050
 	1    0    0    -1
@@
 F 2 "Diode_SMD:D_SOD-123" H 2475 5750 50  0001 C CNN
 F 3 "~" H 2475 5750 50  0001 C CNN
+F 4 "Diodes Inc" H 2475 5750 50  0001 C CNN "MFG Name"
+F 5 " BAV16W-7-F" H 2475 5750 50  0001 C CNN "MFG Part Num"
 	1    2475 5750
 	1    0    0    -1
@@
 F 2 "Resistor_SMD:R_0603_1608Metric" H 1125 6450 50  0001 C CNN
 F 3 "~" H 1125 6450 50  0001 C CNN
+F 4 "Rohm" H 1125 6450 50  0001 C CNN "MFG Name"
+F 5 "ESR03EZPJ102" H 1125 6450 50  0001 C CNN "MFG Part Num"
 	1    1125 6450
 	1    0    0    -1
@@
 F 2 "Resistor_SMD:R_0603_1608Metric" H 1825 6700 50  0001 C CNN
 F 3 "~" H 1825 6700 50  0001 C CNN
+F 4 "Vishay" H 1825 6700 50  0001 C CNN "MFG Name"
+F 5 "RCS06031M00FKEA" H 1825 6700 50  0001 C CNN "MFG Part Num"
 	1    1825 6700
 	1    0    0    -1
@@
 F 2 "Resistor_SMD:R_0603_1608Metric_Pad1.05x0.95mm_HandSolder" H 1825 7400 50  0001 C CNN
 F 3 "~" H 1825 7400 50  0001 C CNN
+F 4 "Rohm" H 1825 7400 50  0001 C CNN "MFG Name"
+F 5 "ESR03EZPJ472" H 1825 7400 50  0001 C CNN "MFG Part Num"
 	1    1825 7400
 	1    0    0    -1
@@
 F 2 "Resistor_SMD:R_0603_1608Metric" H 2975 7050 50  0001 C CNN
 F 3 "~" H 2975 7050 50  0001 C CNN
+F 4 "Rohm" H 2975 7050 50  0001 C CNN "MFG Name"
+F 5 "ESR03EZPJ102" H 2975 7050 50  0001 C CNN "MFG Part Num"
 	1    2975 7050
 	0    -1   -1   0
@@
 	8675 5050 8675 5150
 Wire Wire Line
-	9000 4950 9500 4950
+	9000 4950 9375 4950
 Wire Wire Line
 	9000 4050 9000 4950
@@
 	8675 4250 9200 4250
 Wire Wire Line
-	9500 4650 8675 4650
+	9500 4650 9425 4650
 $Comp
 L 2020-09-12_17-09-47:ISOW7841DWE U2
@@
 L Connector:TestPoint TP4
 U 1 1 5F74616A
-P 9075 4450
-F 0 "TP4" H 9133 4568 50  0000 L CNN
-F 1 "TestPoint" H 9133 4477 50  0000 L CNN
-F 2 "TestPoint:TestPoint_Loop_D1.80mm_Drill1.0mm_Beaded" H 9275 4450 50  0001 C CNN
-F 3 "~" H 9275 4450 50  0001 C CNN
-	1    9075 4450
-	1    0    0    -1
-$EndComp
-Connection ~ 9075 4450
+P 9425 4650
+F 0 "TP4" H 9483 4768 50  0000 L CNN
+F 1 "TestPoint" H 9325 4850 50  0000 L CNN
+F 2 "TestPoint:TestPoint_Loop_D1.80mm_Drill1.0mm_Beaded" H 9625 4650 50  0001 C CNN
+F 3 "~" H 9625 4650 50  0001 C CNN
+	1    9425 4650
+	1    0    0    -1
+$EndComp
 $Comp
 L Device:C_Small C8
@@
 F 2 "Capacitor_SMD:C_0603_1608Metric_Pad1.05x0.95mm_HandSolder" H 7075 3225 50  0001 C CNN
 F 3 "~" H 7075 3225 50  0001 C CNN
+F 4 "Kemet" H 7075 3225 50  0001 C CNN "MFG Name"
+F 5 "C0603C104J4RACTU" H 7075 3225 50  0001 C CNN "MFG Part Num"
 	1    7075 3225
 	1    0    0    -1
@@
 F 2 "Capacitor_SMD:C_0603_1608Metric_Pad1.05x0.95mm_HandSolder" H 7425 3225 50  0001 C CNN
 F 3 "~" H 7425 3225 50  0001 C CNN
+F 4 "Kemet" H 7425 3225 50  0001 C CNN "MFG Name"
+F 5 "C0603C106M9PACTU" H 7425 3225 50  0001 C CNN "MFG Part Num"
 	1    7425 3225
 	1    0    0    -1
@@
 F 2 "Capacitor_SMD:C_0603_1608Metric_Pad1.05x0.95mm_HandSolder" H 9750 3950 50  0001 C CNN
 F 3 "~" H 9750 3950 50  0001 C CNN
+F 4 "Kemet" H 9750 3950 50  0001 C CNN "MFG Name"
+F 5 "C0603C104J4RACTU" H 9750 3950 50  0001 C CNN "MFG Part Num"
 	1    9750 3950
 	1    0    0    -1
@@
 F 2 "Capacitor_SMD:C_0603_1608Metric_Pad1.05x0.95mm_HandSolder" H 10050 3950 50  0001 C CNN
 F 3 "~" H 10050 3950 50  0001 C CNN
+F 4 "Kemet" H 10050 3950 50  0001 C CNN "MFG Name"
+F 5 "C0603C106M9PACTU" H 10050 3950 50  0001 C CNN "MFG Part Num"
 	1    10050 3950
 	1    0    0    -1
@@
 F 2 "Capacitor_SMD:C_0603_1608Metric_Pad1.05x0.95mm_HandSolder" H 11000 4275 50  0001 C CNN
 F 3 "~" H 11000 4275 50  0001 C CNN
+F 4 "Kemet" H 11000 4275 50  0001 C CNN "MFG Name"
+F 5 "C0603C104J4RACTU" H 11000 4275 50  0001 C CNN "MFG Part Num"
 	1    11000 4275
 	0    -1   -1   0
@@
 F 0 "R11" V 10054 5850 50  0000 C CNN
 F 1 "10" V 10145 5850 50  0000 C CNN
-F 2 "Resistor_SMD:R_0603_1608Metric_Pad1.05x0.95mm_HandSolder" H 10250 5850 50  0001 C CNN
+F 2 "Resistor_SMD:R_2512_6332Metric_Pad1.52x3.35mm_HandSolder" H 10250 5850 50  0001 C CNN
 F 3 "~" H 10250 5850 50  0001 C CNN
+F 4 "Vishay" H 10250 5850 50  0001 C CNN "MFG Name"
+F 5 "CRCW251210R0FKEG" H 10250 5850 50  0001 C CNN "MFG Part Num"
 	1    10250 5850
 	0    1    1    0
@@
 F 0 "R10" H 10541 5525 50  0000 R CNN
 F 1 "10" H 10541 5570 50  0001 R CNN
-F 2 "Resistor_SMD:R_0603_1608Metric_Pad1.05x0.95mm_HandSolder" H 10600 5525 50  0001 C CNN
+F 2 "Resistor_SMD:R_2512_6332Metric_Pad1.52x3.35mm_HandSolder" H 10600 5525 50  0001 C CNN
 F 3 "~" H 10600 5525 50  0001 C CNN
+F 4 "Vishay" H 10600 5525 50  0001 C CNN "MFG Name"
+F 5 "CRCW251210R0FKEG" H 10600 5525 50  0001 C CNN "MFG Part Num"
 	1    10600 5525
 	-1   0    0    1
@@
 F 2 "Resistor_SMD:R_0603_1608Metric_Pad1.05x0.95mm_HandSolder" H 10300 5275 50  0001 C CNN
 F 3 "~" H 10300 5275 50  0001 C CNN
+F 4 "Vishay" H 10300 5275 50  0001 C CNN "MFG Name"
+F 5 "CRCW0603120RJNEA" H 10300 5275 50  0001 C CNN "MFG Part Num"
 	1    10300 5275
 	0    -1   -1   0
@@
 	3500 3775 3500 4500
 Wire Wire Line
-	5375 5925 4050 5925
-Wire Wire Line
-	4050 5925 4050 5300
-Wire Wire Line
 	3500 4600 3725 4600
-Wire Wire Line
-	3725 4600 3725 5300
-Wire Wire Line
-	3725 5300 4050 5300
 Wire Wire Line
 	4050 4700 3500 4700
@@
 F 0 "R8" H 9200 1950 50  0000 R CNN
 F 1 "4k7" H 9250 1850 50  0000 R CNN
-F 2 "Resistor_SMD:R_0603_1608Metric_Pad1.05x0.95mm_HandSolder" V 8980 1900 50  0001 C CNN
+F 2 "Resistor_SMD:R_0805_2012Metric_Pad1.15x1.40mm_HandSolder" V 8980 1900 50  0001 C CNN
 F 3 "~" H 9050 1900 50  0001 C CNN
 F 4 "Y" H 9050 1900 50  0001 C CNN "Fit"
+F 5 "Panasonic" H 9050 1900 50  0001 C CNN "MFG Name"
+F 6 "ERJ-P06J472V" H 9050 1900 50  0001 C CNN "MFG Part Num"
 	1    9050 1900
 	1    0    0    -1
@@
 F 3 "~" H 10200 1550 50  0001 C CNN
 F 4 "Y" V 10200 1550 50  0001 C CNN "Fit"
+F 5 "Rohm" H 10200 1550 50  0001 C CNN "MFG Name"
+F 6 "ESR03EZPJ152" H 10200 1550 50  0001 C CNN "MFG Part Num"
 	1    10200 1550
 	0    1    1    0
@@
 F 3 "" H 9560 1790 60  0000 C CNN
 F 4 "Y" V 9450 2050 50  0001 C CNN "Fit"
-F 5 "Multicomp / Littelfuse" V 9450 2050 50  0001 C CNN "Manufacturer"
+F 5 "Multicomp / Diodes" V 9450 2050 50  0001 C CNN "Manufacturer"
 F 6 "SMAJ6.0A" V 9450 2050 50  0001 C CNN "PartNo"
 	1    9450 2050
@@
 Wire Wire Line
 	9550 2250 10550 2250
+Wire Notes Line
+	1200 3400 1200 4350
+Wire Notes Line
+	1200 4350 2650 4350
+Wire Notes Line
+	2650 4350 2650 3400
+Wire Notes Line
+	2650 3400 1200 3400
+Text Notes 1225 3350 0    50   ~ 0
+Voltage Regulator
+Wire Notes Line
+	4525 5475 4525 7650
+Wire Notes Line
+	4525 7650 500  7650
+Wire Notes Line
+	500  7650 500  5475
+Wire Notes Line
+	500  5475 4525 5475
+Text Notes 650  5375 0    50   ~ 0
+Continuity (NC) Check
+Wire Wire Line
+	3725 5400 4950 5400
+Wire Wire Line
+	4950 5400 4950 5925
+Wire Wire Line
+	4950 5925 5375 5925
+Wire Wire Line
+	3725 4600 3725 5400
+Connection ~ 9425 4650
+Wire Wire Line
+	9425 4650 8675 4650
+$Comp
+L Connector:TestPoint TP5
+U 1 1 5F9E5816
+P 9375 4950
+F 0 "TP5" H 9433 5068 50  0000 L CNN
+F 1 "TestPoint" H 9275 5150 50  0000 L CNN
+F 2 "TestPoint:TestPoint_Loop_D1.80mm_Drill1.0mm_Beaded" H 9575 4950 50  0001 C CNN
+F 3 "~" H 9575 4950 50  0001 C CNN
+	1    9375 4950
+	-1   0    0    1
+$EndComp
+Connection ~ 9375 4950
+Wire Wire Line
+	9375 4950 9500 4950
 $EndSCHEMATC

Commit message: Aisler fab submit
Parts:
- C0: MFG Name (none) -> Panasonic; MFG Part Num (none) -> ECQU2A104ML
- C1, C2: MFG Name (none) -> Vishay; MFG Part Num (none) -> BFC233660473
- CP2: symbol pwrcon-rescue:CAP_POL-baseunit -> Device:CP_Small; MFG Name (none) -> Kemet; MFG Part Num (none) -> T495V157M010ATE150
- D2: MFG Name (none) -> Diodes Inc; MFG Part Num (none) -> SMAJ6.0A
- DR2: symbol pwrcon-rescue:LED_18-baseunit -> Device:LED; MFG Name (none) -> Osram; MFG Part Num (none) -> LS Q976-NR-1
- LC1: symbol pwrcon-rescue:TRANSFORMER_ISOLATED_1_0-baseunit -> pwrcon:choke
- PS1: MFG Name (none) -> Meanwell; MFG Part Num (none) -> IRM-01-5
- RV1: symbol pwrcon-rescue:VARISTOR-baseunit -> Device:Varistor; MFG Name (none) -> Wurth Elektronik; MFG Part Num (none) -> 820572711
- U5, U6: MFG Name (none) -> TI; MFG Part Num (none) -> SN74LV1T34DBVR
- U7: MFG Name (none) -> Microchip; MFG Part Num (none) -> MIC5219-3.3YMM
Connections:
- net GND: now also DR2.1 (K); no longer DR2.2, J6.3 (Pin_3)
- net RS485_RXD: now also J8.3 (Pin_3); no longer J8.2 (Pin_2)
- net RS485_TXD: now also J8.2 (Pin_2); no longer J8.3 (Pin_3)
- net at R9.1: now also DR2.2 (A); no longer DR2.1
Changed lines of the file:
@@
 Wire Wire Line
 	6900 1550 6900 1850
-Wire Wire Line
-	6900 2250 6900 2450
 Text Label 2250 2650 0    50   ~ 0
 LIVE
@@
 	6150 2050 5850 2050
 $Comp
-L pwrcon-rescue:VARISTOR-baseunit RV1
+L Device:Varistor RV1
 U 1 1 5BE08674
-P 7000 1950
-F 0 "RV1" H 7300 1900 50  0000 C CNN
-F 1 "275V" H 7400 1780 60  0000 R BNN
-F 2 "Varistor:RV_Disc_D7mm_W4mm_P5mm" H 7400 1780 60  0001 C CNN
-F 3 "" H 7400 1780 60  0000 C CNN
-F 4 "Y" H 7000 1950 50  0001 C CNN "Fit"
-F 5 "Wurth Elektronik" H 7000 1950 50  0001 C CNN "Manufacturer"
-F 6 "820572711" H 7000 1950 50  0001 C CNN "PartNo"
-	1    7000 1950
+P 6900 2000
+F 0 "RV1" H 7075 2075 50  0000 C CNN
+F 1 "275V" H 7200 1850 60  0000 R BNN
+F 2 "Varistor:RV_Disc_D7mm_W4mm_P5mm" H 7300 1830 60  0001 C CNN
+F 3 "" H 7300 1830 60  0000 C CNN
+F 4 "Y" H 6900 2000 50  0001 C CNN "Fit"
+F 5 "Wurth Elektronik" H 6900 2000 50  0001 C CNN "Manufacturer"
+F 6 "820572711" H 6900 2000 50  0001 C CNN "PartNo"
+F 7 "Wurth Elektronik" H 6900 2000 50  0001 C CNN "MFG Name"
+F 8 "820572711" H 6900 2000 50  0001 C CNN "MFG Part Num"
+	1    6900 2000
 	-1   0    0    -1
 $EndComp
@@
 F 5 "Panasonic" H 4350 2000 50  0001 C CNN "Manufacturer"
 F 6 "ECQU2A104ML" H 4350 2000 50  0001 C CNN "PartNo"
+F 7 "Panasonic" H 4350 2000 50  0001 C CNN "MFG Name"
+F 8 "ECQU2A104ML" H 4350 2000 50  0001 C CNN "MFG Part Num"
 	1    4350 2000
 	-1   0    0    1
@@
 F 5 "Vishay" H 6150 1700 50  0001 C CNN "Manufacturer"
 F 6 "BFC233660473" H 6150 1700 50  0001 C CNN "PartNo"
+F 7 "Vishay" H 6150 1700 50  0001 C CNN "MFG Name"
+F 8 "BFC233660473" H 6150 1700 50  0001 C CNN "MFG Part Num"
 	1    6150 1700
 	-1   0    0    1
@@
 F 5 "Y" H 6150 2300 50  0001 C CNN "Fit"
 F 6 "Vishay" H 6150 2300 50  0001 C CNN "Manufacturer"
+F 7 "Vishay" H 6150 2300 50  0001 C CNN "MFG Name"
+F 8 "BFC233660473" H 6150 2300 50  0001 C CNN "MFG Part Num"
 	1    6150 2300
 	-1   0    0    1
@@
 NEUTRAL
 $Comp
-L pwrcon-rescue:TRANSFORMER_ISOLATED_1_0-baseunit LC1
+L pwrcon:choke LC1
 U 1 1 5BFC18B6
 P 5350 1850
@@
 Connection ~ 3775 6400
 Wire Wire Line
-	3775 6500 3775 7025
-Connection ~ 3775 6500
-Wire Wire Line
 	4350 7050 4350 7225
 Wire Wire Line
 	3225 7050 4350 7050
-Wire Wire Line
-	4150 7225 4150 7025
-Wire Wire Line
-	4150 7025 3775 7025
 $Comp
 L Connector_Generic:Conn_01x04 J6
@@
 F 2 "SN74LV1T34DBVR:SN74LV1T34DBVR" H 4750 4640 60  0001 C CNN
 F 3 "" H 4750 4700 60  0000 C CNN
+F 4 "TI" H 4750 4700 50  0001 C CNN "MFG Name"
+F 5 "SN74LV1T34DBVR" H 4750 4700 50  0001 C CNN "MFG Part Num"
 	1    4750 4700
 	1    0    0    -1
@@
 F 2 "SN74LV1T34DBVR:SN74LV1T34DBVR" H 6175 5865 60  0001 C CNN
 F 3 "" H 6175 5925 60  0000 C CNN
+F 4 "TI" H 6175 5925 50  0001 C CNN "MFG Name"
+F 5 "SN74LV1T34DBVR" H 6175 5925 50  0001 C CNN "MFG Part Num"
 	1    6175 5925
 	-1   0    0    1
@@
 $EndComp
 Wire Wire Line
-	5450 3775 3500 3775
-Wire Wire Line
-	3500 3775 3500 4500
-Wire Wire Line
-	3500 4600 3725 4600
+	5450 3775 3600 3775
 Wire Wire Line
 	4050 4700 3500 4700
-Text Label 3725 4600 0    50   ~ 0
+Text Label 3500 4500 1    50   ~ 0
 RS485_RXD
-Text Label 3500 4500 0    50   ~ 0
+Text Label 3500 4600 3    50   ~ 0
 RS485_TXD
 Text Label 1025 7050 1    50   ~ 0
@@
 F 2 "Package_SO:MSOP-8_3x3mm_P0.65mm" H 1850 4125 50  0001 C CNN
 F 3 "http://ww1.microchip.com/downloads/en/DeviceDoc/MIC5219-500mA-Peak-Output-LDO-Regulator-DS20006021A.pdf" H 1850 3800 50  0001 C CNN
+F 4 "Microchip" H 1850 3800 50  0001 C CNN "MFG Name"
+F 5 "MIC5219-3.3YMM" H 1850 3800 50  0001 C CNN "MFG Part Num"
 	1    1850 3800
 	1    0    0    -1
@@
 	2150 4100 2325 4100
 $Comp
-L pwrcon-rescue:LED_18-baseunit DR2
+L Device:LED DR2
 U 1 1 5BE0866A
-P 10750 1850
-F 0 "DR2" V 10650 1725 50  0000 C CNN
-F 1 "LSQ976-Z Red" H 10450 1475 60  0000 L BNN
-F 2 "LED_SMD:LED_0603_1608Metric_Pad1.05x0.95mm_HandSolder" H 10920 1850 60  0001 C CNN
-F 3 "" H 10920 1850 60  0000 C CNN
-F 4 "Y" V 10750 1850 50  0001 C CNN "Fit"
-F 5 "Osram" V 10750 1850 50  0001 C CNN "Manufacturer"
-F 6 "LS Q976-NR-1" V 10750 1850 50  0001 C CNN "PartNo"
-	1    10750 1850
-	0    1    1    0
+P 10550 1900
+F 0 "DR2" V 10450 1775 50  0000 C CNN
+F 1 "LSQ976-Z Red" H 10250 1525 60  0000 L BNN
+F 2 "LED_SMD:LED_0603_1608Metric_Pad1.05x0.95mm_HandSolder" H 10720 1900 60  0001 C CNN
+F 3 "" H 10720 1900 60  0000 C CNN
+F 4 "Y" V 10550 1900 50  0001 C CNN "Fit"
+F 5 "Osram" V 10550 1900 50  0001 C CNN "Manufacturer"
+F 6 "LS Q976-NR-1" V 10550 1900 50  0001 C CNN "PartNo"
+F 7 "Osram" H 10550 1900 50  0001 C CNN "MFG Name"
+F 8 "LS Q976-NR-1" H 10550 1900 50  0001 C CNN "MFG Part Num"
+	1    10550 1900
+	0    -1   -1   0
 $EndComp
 Connection ~ 9050 1550
@@
 Connection ~ 8100 2250
 $Comp
-L pwrcon-rescue:CAP_POL-baseunit CP2
+L Device:CP_Small CP2
 U 1 1 5BE0866C
-P 8000 1750
-F 0 "CP2" H 8300 1750 50  0000 C CNN
-F 1 "150uF" H 8250 1600 60  0000 L BNN
-F 2 "Capacitor_Tantalum_SMD:CP_EIA-7343-20_Kemet-V_Pad2.25x2.55mm_HandSolder" H 8290 1590 60  0001 C CNN
-F 3 "" H 8290 1590 60  0000 C CNN
-F 4 "Y" H 8000 1750 50  0001 C CNN "Fit"
-F 5 "AVX / Kemet" H 8000 1750 50  0001 C CNN "Manufacturer"
-F 6 "TRJD157K010R0150 / T495V157M010ATE150 " H 8000 1750 50  0001 C CNN "PartNo"
-	1    8000 1750
+P 8100 1750
+F 0 "CP2" H 8250 1825 50  0000 C CNN
+F 1 "150uF" H 8175 1600 60  0000 L BNN
+F 2 "Capacitor_Tantalum_SMD:CP_EIA-7343-20_Kemet-V_Pad2.25x2.55mm_HandSolder" H 8390 1590 60  0001 C CNN
+F 3 "" H 8390 1590 60  0000 C CNN
+F 4 "Y" H 8100 1750 50  0001 C CNN "Fit"
+F 5 "AVX / Kemet" H 8100 1750 50  0001 C CNN "Manufacturer"
+F 6 "TRJD157K010R0150 / T495V157M010ATE150 " H 8100 1750 50  0001 C CNN "PartNo"
+F 7 "Kemet" H 8100 1750 50  0001 C CNN "MFG Name"
+F 8 "T495V157M010ATE150" H 8100 1750 50  0001 C CNN "MFG Part Num"
+	1    8100 1750
 	1    0    0    -1
 $EndComp
@@
 F 5 "Multicomp / Diodes" V 9450 2050 50  0001 C CNN "Manufacturer"
 F 6 "SMAJ6.0A" V 9450 2050 50  0001 C CNN "PartNo"
+F 7 "Diodes Inc" H 9450 2050 50  0001 C CNN "MFG Name"
+F 8 "SMAJ6.0A" H 9450 2050 50  0001 C CNN "MFG Part Num"
 	1    9450 2050
 	0    -1   -1   0
@@
 Text Notes 9850 2490 0    84   ~ 17
 Power LED
-Wire Wire Line
-	8100 2050 8100 2250
 Wire Wire Line
 	8100 1550 8100 1650
@@
 F 2 "Converter_ACDC:Converter_ACDC_MeanWell_IRM-02-xx_THT" H 7500 1350 50  0001 C CNN
 F 3 "https://www.meanwell.com/Upload/PDF/IRM-02/IRM-02-SPEC.PDF" H 7900 1300 50  0001 C CNN
+F 4 "Meanwell" H 7500 1650 50  0001 C CNN "MFG Name"
+F 5 "IRM-01-5" H 7500 1650 50  0001 C CNN "MFG Part Num"
 	1    7500 1650
 	1    0    0    -1
@@
 Wire Wire Line
 	4950 5925 5375 5925
-Wire Wire Line
-	3725 4600 3725 5400
 Connection ~ 9425 4650
 Wire Wire Line
@@
 Wire Wire Line
 	9375 4950 9500 4950
+Wire Wire Line
+	3500 4600 3600 4600
+Wire Wire Line
+	3600 4600 3600 3775
+Wire Wire Line
+	3500 4500 3725 4500
+Wire Wire Line
+	3725 4500 3725 5400
+Wire Wire Line
+	8100 1850 8100 2250
+Wire Wire Line
+	6900 2150 6900 2450
 $EndSCHEMATC
